Commit message: model color, limits

File: src/ah_urdf/urdf/ability_hand_right_large_gazebo.xacro (robot description, xacro)
@@ -15,5 +15,5 @@
           <command_interface name="position">
             <param name="min">0.0</param>
-            <param name="max">2.0</param>
+            <param name="max">1.85</param>
           </command_interface>
           <state_interface name="position">
@@ -27,5 +27,5 @@
           <command_interface name="position">
             <param name="min">0.0</param>
-            <param name="max">2.0</param>
+            <param name="max">1.85</param>
           </command_interface>
           <state_interface name="position">
@@ -39,5 +39,5 @@
           <command_interface name="position">
             <param name="min">0.0</param>
-            <param name="max">2.0</param>
+            <param name="max">1.85</param>
           </command_interface>
           <state_interface name="position">
@@ -51,5 +51,5 @@
           <command_interface name="position">
             <param name="min">0.0</param>
-            <param name="max">2.0</param>
+            <param name="max">1.90</param>
           </command_interface>
           <state_interface name="position">

File: src/ah_urdf/urdf/ability_hand_right_large_macro.xacro (robot description, xacro)
@@ -2,4 +2,10 @@
 <robot xmlns:xacro="http://www.ros.org/wiki/xacro" name="ability_hand_macro">
    <xacro:include filename="$(find ah_urdf)/urdf/ability_hand_right_large_gazebo.xacro"/>
+   <material name="ability_hand_gray">
+      <color rgba="0.55 0.55 0.55 1.0" />
+   </material>
+   <material name="ability_hand_black">
+      <color rgba="0.1 0.1 0.1 1.0" />
+   </material>
    <xacro:macro name="ability_hand_right_large" params="prefix:='' parent:='base_link' sim_gz:='false' *origin">
     <joint name="${prefix}mount_joint" type="fixed">
@@ -14,4 +20,5 @@
                 <mesh filename="file://$(find ah_urdf)/models/wristmesh.STL" />
              </geometry>
+             <material name="ability_hand_gray" />
           </visual>
           <inertial>
@@ -25,4 +32,5 @@
                 <mesh filename="file://$(find ah_urdf)/models/FB_palm_ref_MIR.STL" />
              </geometry>
+             <material name="ability_hand_gray" />
           </visual>
           <collision name="palm_mesh_coll">
@@ -44,4 +52,5 @@
                 <mesh filename="file://$(find ah_urdf)/models/idx-F1.STL" />
              </geometry>
+             <material name="ability_hand_black" />
           </visual>
           <collision name="index_mesh_coll_1">
@@ -63,4 +72,5 @@
                 <mesh filename="file://$(find ah_urdf)/models/idx-F2-Lg.STL" />
              </geometry>
+             <material name="ability_hand_black" />
           </visual>
           <collision name="index_mesh_coll_2">
@@ -76,5 +86,5 @@
           <origin xyz="-2.8e-2 -9e-3 9.6e-2" rpy=" 1.672 -1.317 -1.790 " />
           <axis xyz="0 0 1" />
-          <limit lower="0" upper="2.00" effort="6.0" velocity="8.0677777442" />
+          <limit lower="0" upper="1.85" effort="6.0" velocity="8.0677777442" />
           <dynamics damping="0.001" friction="0.001" />
        </joint>
@@ -141,4 +151,5 @@
                 <mesh filename="file://$(find ah_urdf)/models/idx-F1.STL" />
              </geometry>
+             <material name="ability_hand_black" />
           </visual>
           <collision name="middle_mesh_coll_1">
@@ -160,4 +171,5 @@
                 <mesh filename="file://$(find ah_urdf)/models/idx-F2-Lg.STL" />
              </geometry>
+             <material name="ability_hand_black" />
           </visual>
           <collision name="middle_mesh_coll_2">
@@ -172,5 +184,5 @@
           <child link="${prefix}middle_L1" />
           <origin xyz=" -0.008 -0.012 0.099 " rpy=" 1.513 -1.322 -1.558 " />
-          <limit lower="0" upper="2.00" effort="6.0" velocity="8.0677777442" />
+          <limit lower="0" upper="1.85" effort="6.0" velocity="8.0677777442" />
           <dynamics damping="0.001" friction="0.001" />
           <axis xyz="0 0 1" />
@@ -238,4 +250,5 @@
                 <mesh filename="file://$(find ah_urdf)/models/idx-F1.STL" />
              </geometry>
+             <material name="ability_hand_black" />
           </visual>
           <collision name="ring_mesh_coll_1">
@@ -257,4 +270,5 @@
                 <mesh filename="file://$(find ah_urdf)/models/idx-F2-Lg.STL" />
              </geometry>
+             <material name="ability_hand_black" />
           </visual>
           <collision name="ring_mesh_coll_2">
@@ -269,5 +283,5 @@
           <child link="${prefix}ring_L1" />
           <origin xyz=" 0.012 -0.010 0.097 " rpy=" 1.361 -1.315 -1.330 " />
-          <limit lower="0" upper="2.00" effort="6.0" velocity="8.0677777442" />
+          <limit lower="0" upper="1.85" effort="6.0" velocity="8.0677777442" />
           <dynamics damping="0.001" friction="0.001" />
           <axis xyz="0 0 1" />
@@ -335,4 +349,5 @@
                 <mesh filename="file://$(find ah_urdf)/models/idx-F1.STL" />
              </geometry>
+             <material name="ability_hand_black" />
           </visual>
           <collision name="pinky_mesh_coll_1">
@@ -354,4 +369,5 @@
                 <mesh filename="file://$(find ah_urdf)/models/idx-F2.STL" />
              </geometry>
+             <material name="ability_hand_black" />
           </visual>
           <collision name="pinky_mesh_coll_2">
@@ -366,5 +382,5 @@
           <child link="${prefix}pinky_L1" />
           <origin xyz=" 0.031 -0.007 0.091 " rpy=" 1.410 -1.315 -1.313 " />
-          <limit lower="0" upper="2.00" effort="6.0" velocity="8.0677777442" />
+          <limit lower="0" upper="1.90" effort="6.0" velocity="8.0677777442" />
           <dynamics damping="0.001" friction="0.001" />
           <axis xyz="0 0 1" />
@@ -432,4 +448,5 @@
                 <mesh filename="file://$(find ah_urdf)/models/thumb-F1-MIR.STL" />
              </geometry>
+             <material name="ability_hand_black" />
           </visual>
           <collision name="thumb_coll_mesh_1">
@@ -451,4 +468,5 @@
                 <mesh filename="file://$(find ah_urdf)/models/thumb-F2-right.STL" />
              </geometry>
+             <material name="ability_hand_black" />
           </visual>
           <collision name="thumb_hull_mesh_2">
